File: seg7.kicad_sch (KiCad schematic)
At the start: 33 parts, among them U1 74HC595, U2 74HC595, U3 TD62083, U4 TD62083, U5 74HC595, U6 TD62083

Commit message: update
Parts:
- added Q1, Q2, Q3: 2SA1037, Package_TO_SOT_SMD:SOT-23, symbol Transistor_BJT:BC807
- added R25, R26, R27: 1.2K, Resistor_SMD:R_0603_1608Metric_Pad0.98x0.95mm_HandSolder, symbol Device:R
Connections:
- net +5V: now also Q1.2 (E), Q2.2 (E), Q3.2 (E); no longer D1.1 (Pin_1), D2.1 (Pin_1), D3.1 (Pin_1)
- net GND: no longer D1.6 (Pin_6), D2.6 (Pin_6), D3.6 (Pin_6)
- new net: Q2.1 (B), R25.2
- new net: Q1.1 (B), R26.2
- new net: Q3.1 (B), R27.2
- new net PWR1: D1.1 (Pin_1), D1.6 (Pin_6), Q2.3 (C)
- new net PWR2: D2.1 (Pin_1), D2.6 (Pin_6), Q1.3 (C)
- new net PWR3: D3.1 (Pin_1), D3.6 (Pin_6), Q3.3 (C)
- new net SIG1: R25.1
- new net SIG2: R26.1
- new net SIG3: R27.1
